Commit message: feat: add LiDAR filtering, utility nodes, and twist mux

File: src/panda_description/urdf/gazebo.xacro (robot description, xacro)
@@ -67,29 +67,29 @@
     <gazebo reference="laser_link">
         <sensor name="lidar" type="gpu_lidar">
-        <always_on>true</always_on>
-        <visualize>true</visualize>
-        <topic>scan</topic>
-        <update_rate>5</update_rate>
-        <gz_frame_id>laser_link</gz_frame_id>
-        <lidar>
-            <scan>
-            <horizontal>
-                <samples>360</samples>
-                <resolution>1.00000</resolution>
-                <min_angle>0.000000</min_angle>
-                <max_angle>6.280000</max_angle>
-            </horizontal>
-            </scan>
-            <range>
-            <min>0.120000</min>
-            <max>12.0</max>
-            <resolution>0.02</resolution>
-            </range>
-            <noise>
-            <type>gaussian</type>
-            <mean>0.0</mean>
-            <stddev>0.01</stddev>
-            </noise>
-        </lidar>
+            <always_on>true</always_on>
+            <visualize>true</visualize>
+            <topic>scan</topic>
+            <update_rate>10</update_rate>
+            <gz_frame_id>laser_link</gz_frame_id>
+            <lidar>
+                <scan>
+                    <horizontal>
+                        <samples>360</samples>
+                        <resolution>1.00000</resolution>
+                        <min_angle>0.000000</min_angle>
+                        <max_angle>6.283185</max_angle>
+                    </horizontal>
+                </scan>
+                <range>
+                    <min>0.120000</min>
+                    <max>12.0</max>
+                    <resolution>0.02</resolution>
+                </range>
+                <noise>
+                    <type>gaussian</type>
+                    <mean>0.0</mean>
+                    <stddev>0.01</stddev>
+                </noise>
+            </lidar>
         </sensor>
     </gazebo>

File: src/panda_description/urdf/panda.urdf.xacro (robot description, xacro)
@@ -220,5 +220,5 @@
   </link>
   <joint name="laser_joint" type="fixed">
-    <origin xyz="0 0 0.2186" rpy="0 0 0" />
+    <origin xyz="0.175 0 0.2186" rpy="0 0 0" />
     <parent link="base_link" />
     <child link="laser_link" />
